Commit message: ROS 1 -> ROS 2 Humble Migration komplett: URDF, Launch-Files, Scripts, MoveIt2, RViz Konfiguration

File: urdf/ur5_rg2.urdf (robot description, URDF)
Before this commit: robot ur5_rg2, 11 links, 10 joints
Links:
- added link world
- link base_link: mass None -> 4.210389694173812; geometry collision mesh filename=package://ur5_rg2_ign/ur5_rg2/meshes/collision/ur5/base.stl; visual mesh filename=package://ur5_rg2_ign/ur5_rg2/meshes/visual/ur5/base.dae
- link forearm_link: mass None -> 2.275; geometry collision mesh filename=package://ur5_rg2_ign/ur5_rg2/meshes/collision/ur5/forearm.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; visual mesh filename=package://ur5_rg2_ign/ur5_rg2/meshes/visual/ur5/forearm.dae
- link rg2_hand: mass None -> 0.5; geometry collision mesh filename=package://ur5_rg2_ign/ur5_rg2/meshes/collision/rg2/hand.stl; visual mesh filename=package://ur5_rg2_ign/ur5_rg2/meshes/visual/rg2/hand.dae
- link rg2_leftfinger: mass None -> 0.1; geometry collision mesh filename=package://ur5_rg2_ign/ur5_rg2/meshes/collision/rg2/finger.s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; visual mesh filename=package://ur5_rg2_ign/ur5_rg2/meshes/visual/rg2/finger.dae
- link rg2_rightfinger: mass None -> 0.1; geometry collision mesh filename=package://ur5_rg2_ign/ur5_rg2/meshes/collision/rg2/finger.s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; visual mesh filename=package://ur5_rg2_ign/ur5_rg2/meshes/visual/rg2/finger.dae
- link shoulder_link: mass None -> 2.6078628081050645; geometry collision mesh filename=package://ur5_rg2_ign/ur5_rg2/meshes/collision/ur5/shoulder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; visual mesh filename=package://ur5_rg2_ign/ur5_rg2/meshes/visual/ur5/shoulder.dae
- link tool0: mass None -> 0.001
- link upper_arm_link: mass None -> 9.034556202946057; geometry collision mesh filename=package://ur5_rg2_ign/ur5_rg2/meshes/collision/ur5/upperarm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; visual mesh filename=package://ur5_rg2_ign/ur5_rg2/meshes/visual/ur5/upperarm.dae
- link wrist_1_link: mass None -> 0.8652783044597422; geometry collision mesh filename=package://ur5_rg2_ign/ur5_rg2/meshes/collision/ur5/wrist1.s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; visual mesh filename=package://ur5_rg2_ign/ur5_rg2/meshes/visual/ur5/wrist1.dae
- link wrist_2_link: mass None -> 1.219; geometry collision mesh filename=package://ur5_rg2_ign/ur5_rg2/meshes/collision/ur5/wrist2.s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; visual mesh filename=package://ur5_rg2_ign/ur5_rg2/meshes/visual/ur5/wrist2.dae
- link wrist_3_link: mass None -> 0.1879; geometry collision mesh filename=package://ur5_rg2_ign/ur5_rg2/meshes/collision/ur5/wrist3.s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; visual mesh filename=package://ur5_rg2_ign/ur5_rg2/meshes/visual/ur5/wrist3.dae
Joints:
- added joint world_joint: type fixed, parent world, child base_link, origin xyz=0 0 0 rpy=0 0 0
- joint rg2_finger_joint2: mimic joint=panda_finger_joint1 -> joint=rg2_finger_joint1 multiplier=1.0 offset=0.0

Commit message: Aktueller Stand: neue RG2 Meshes, GUI Fix, Greifposition kalibriert

File: urdf/ur5_rg2.urdf (robot description, URDF)
Before this commit: robot ur5_rg2, 12 links, 11 joints
Joints:
- joint ur5_hand_joint: origin xyz=0 0.0823 0 rpy=1.570796325 0 1.570796325 -> xyz=0 0 0 rpy=1.570796325 0 1.570796325

Commit message: Mimic Plugin integriert, parallele Finger, Greifposition nah am Würfel

File: urdf/ur5_rg2.urdf (robot description, URDF)
Before this commit: robot ur5_rg2, 12 links, 11 joints
Joints:
- joint rg2_finger_joint1: axis 0 0 1 -> 1 0 0; limit lower=0.0 upper=1.18 effort=10.6 velocity=1.57 -> lower=-0.5 upper=0.5 effort=10.6 velocity=1.57; origin xyz=0.105 0.017 0 rpy=0 0 0 -> xyz=0 0.05 0 rpy=0 0 0
- joint rg2_finger_joint2: axis 0 0 -1 -> -1 0 0; limit lower=0.0 upper=1.18 effort=10.6 velocity=1.57 -> lower=-0.5 upper=0.5 effort=10.6 velocity=1.57; origin xyz=0.105 -0.017 0 rpy=0 0 0 -> xyz=0 -0.05 0 rpy=0 0 0
- joint ur5_hand_joint: origin xyz=0 0 0 rpy=1.570796325 0 1.570796325 -> xyz=0 0.0823 0 rpy=1.570796325 0 1.570796325

Commit message: Finger-Joints korrekt ausgerichtet - parallele Greifbewegung

File: urdf/ur5_rg2.urdf (robot description, URDF)
Before this commit: robot ur5_rg2, 12 links, 11 joints
Joints:
- joint rg2_finger_joint1: axis 1 0 0 -> 0 1 0; origin xyz=0 0.05 0 rpy=0 0 0 -> xyz=0.105 0.017 0 rpy=0 0 0
- joint rg2_finger_joint2: axis -1 0 0 -> 0 -1 0; origin xyz=0 -0.05 0 rpy=0 0 0 -> xyz=0.105 -0.017 0 rpy=0 0 0

Commit message: Finger-Achse X mit RPY Rotation - weitere Versuche

File: urdf/ur5_rg2.urdf (robot description, URDF)
Before this commit: robot ur5_rg2, 12 links, 11 joints
Joints:
- joint rg2_finger_joint1: axis 0 1 0 -> 1 0 0; origin xyz=0.105 0.017 0 rpy=0 0 0 -> xyz=0.105 0.017 0 rpy=0 1.570796325 0
- joint rg2_finger_joint2: axis 0 -1 0 -> -1 0 0; origin xyz=0.105 -0.017 0 rpy=0 0 0 -> xyz=0.105 -0.017 0 rpy=0 1.570796325 0

Commit message: Finger original Montage wiederhergestellt - Scherenöffnung Problem bleibt

File: urdf/ur5_rg2.urdf (robot description, URDF)
Before this commit: robot ur5_rg2, 12 links, 11 joints
Joints:
- joint rg2_finger_joint1: axis 1 0 0 -> 0 0 1; limit lower=-0.5 upper=0.5 effort=10.6 velocity=1.57 -> lower=0.0 upper=1.18 effort=10.6 velocity=1.57; origin xyz=0.105 0.017 0 rpy=0 1.570796325 0 -> xyz=0.105 0.017 0 rpy=0 0 0
- joint rg2_finger_joint2: axis -1 0 0 -> 0 0 -1; limit lower=-0.5 upper=0.5 effort=10.6 velocity=1.57 -> lower=0.0 upper=1.18 effort=10.6 velocity=1.57; origin xyz=0.105 -0.017 0 rpy=0 1.570796325 0 -> xyz=0.105 -0.017 0 rpy=0 0 0

Commit message: Würfel Reibung erhöht, Masse 0.5kg

File: urdf/ur5_rg2.urdf (robot description, URDF)
Before this commit: robot ur5_rg2, 12 links, 11 joints
Joints:
- joint rg2_finger_joint1: limit lower=0.0 upper=1.18 effort=10.6 velocity=1.57 -> lower=0.0 upper=1.18 effort=2.0 velocity=0.3

Commit message: Parallelgreifer funktioniert - Montage noch zu klären

File: urdf/ur5_rg2.urdf (robot description, URDF)
Before this commit: robot ur5_rg2, 12 links, 11 joints
Links:
- removed link rg2_hand
- removed link rg2_leftfinger
- removed link rg2_rightfinger
- added link finger_1_finger_tip, mass 0.001; collision mesh filename=package://ur5_rg2_ign/ur5_rg2/meshes/visual/rg2/finger_tip.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; visual mesh filename=package://ur5_rg2_ign/ur5_rg2/meshes/visual/rg2/finger_tip.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
- added link finger_1_flex_finger, mass 0.001; collision mesh filename=package://ur5_rg2_ign/ur5_rg2/meshes/visual/rg2/flex_finger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; visual mesh filename=package://ur5_rg2_ign/ur5_rg2/meshes/visual/rg2/flex_finger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
- added link finger_1_moment_arm, mass 0.001; collision mesh filename=package://ur5_rg2_ign/ur5_rg2/meshes/visual/rg2/moment_arm.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; visual mesh filename=package://ur5_rg2_ign/ur5_rg2/meshes/visual/rg2/moment_arm.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
- added link finger_1_origin, mass 0.001
- added link finger_1_truss_arm, mass 0.001; collision mesh filename=package://ur5_rg2_ign/ur5_rg2/meshes/visual/rg2/truss_arm.s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; visual mesh filename=package://ur5_rg2_ign/ur5_rg2/meshes/visual/rg2/truss_arm.s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
- added link finger_2_finger_tip, mass 0.001; collision mesh filename=package://ur5_rg2_ign/ur5_rg2/meshes/visual/rg2/finger_tip.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; visual mesh filename=package://ur5_rg2_ign/ur5_rg2/meshes/visual/rg2/finger_tip.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
- added link finger_2_flex_finger, mass 0.001; collision mesh filename=package://ur5_rg2_ign/ur5_rg2/meshes/visual/rg2/flex_finger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; visual mesh filename=package://ur5_rg2_ign/ur5_rg2/meshes/visual/rg2/flex_finger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
- added link finger_2_moment_arm, mass 0.001; collision mesh filename=package://ur5_rg2_ign/ur5_rg2/meshes/visual/rg2/moment_arm.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; visual mesh filename=package://ur5_rg2_ign/ur5_rg2/meshes/visual/rg2/moment_arm.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
- added link finger_2_origin, mass 0.001
- added link finger_2_truss_arm, mass 0.001; collision mesh filename=package://ur5_rg2_ign/ur5_rg2/meshes/visual/rg2/truss_arm.s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; visual mesh filename=package://ur5_rg2_ign/ur5_rg2/meshes/visual/rg2/truss_arm.s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
- added link gripper_body, mass 0.65; collision mesh filename=package://ur5_rg2_ign/ur5_rg2/meshes/visual/rg2/body.stl; visual mesh filename=package://ur5_rg2_ign/ur5_rg2/meshes/visual/rg2/body.stl
- added link gripper_bracket, mass 0.09; collision mesh filename=package://ur5_rg2_ign/ur5_rg2/meshes/visual/rg2/single_brac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; visual mesh filename=package://ur5_rg2_ign/ur5_rg2/meshes/visual/rg2/single_brac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
Joints:
- removed joint ur5_hand_joint
- added joint finger_1_finger_tip_joint: type revolute, parent finger_1_truss_arm, child finger_1_finger_tip, origin xyz=-0.0256 0.0 0.04868 rpy=0.0 0.772 0.0, axis 0 -1 0, limit lower=0.0 upper=1.3 effort=10.0 velocity=50.0, mimic joint=rg2_finger_joint1 multiplier=1 offset=0
- added joint finger_1_flex_finger_joint: type fixed, parent finger_1_finger_tip, child finger_1_flex_finger, origin xyz=0.03059 0.0 0.0172 rpy=0 0 0
- added joint finger_1_origin_joint: type fixed, parent gripper_body, child finger_1_origin, origin xyz=0 0 0 rpy=0 0 0
- added joint finger_1_truss_arm_joint: type revolute, parent finger_1_origin, child finger_1_truss_arm, origin xyz=-0.0075 0.0 0.0715 rpy=0.0 -0.772 0.0, axis 0 1 0, limit lower=0.0 upper=1.3 effort=10.0 velocity=50.0, mimic joint=rg2_finger_joint1 multiplier=1 offset=0
- added joint finger_2_finger_tip_joint: type revolute, parent finger_2_truss_arm, child finger_2_finger_tip, origin xyz=-0.0256 0.0 0.04868 rpy=0.0 0.772 0.0, axis 0 -1 0, limit lower=0.0 upper=1.3 effort=10.0 velocity=50.0, mimic joint=rg2_finger_joint1 multiplier=1 offset=0
- added joint finger_2_flex_finger_joint: type fixed, parent finger_2_finger_tip, child finger_2_flex_finger, origin xyz=0.03059 0.0 0.0172 rpy=0 0 0
- added joint finger_2_origin_joint: type fixed, parent gripper_body, child finger_2_origin, origin xyz=0 0 0 rpy=0 0 3.14159265
- added joint finger_2_truss_arm_joint: type revolute, parent finger_2_origin, child finger_2_truss_arm, origin xyz=-0.0075 0.0 0.0715 rpy=0.0 -0.772 0.0, axis 0 1 0, limit lower=0.0 upper=1.3 effort=10.0 velocity=50.0, mimic joint=rg2_finger_joint1 multiplier=1 offset=0
- added joint gripper_body_joint: type fixed, parent gripper_bracket, child gripper_body, origin xyz=0.0 0.0 0.05 rpy=0 0 0
- added joint gripper_bracket_joint: type fixed, parent wrist_3_link, child gripper_bracket, origin xyz=0 0 0.05 rpy=0 0 0
- joint rg2_finger_joint1: axis 0 0 1 -> 0 1 0; child rg2_leftfinger -> finger_1_moment_arm; limit lower=0.0 upper=1.18 effort=2.0 velocity=0.3 -> lower=0.0 upper=1.3 effort=10.0 velocity=50.0; origin xyz=0.105 0.017 0 rpy=0 0 0 -> xyz=-0.017 0.0 0.055 rpy=0.0 -0.772 0.0; parent rg2_hand -> finger_1_origin
- joint rg2_finger_joint2: axis 0 0 -1 -> 0 1 0; child rg2_rightfinger -> finger_2_moment_arm; limit lower=0.0 upper=1.18 effort=10.6 velocity=1.57 -> lower=0.0 upper=1.3 effort=10.0 velocity=50.0; mimic joint=rg2_finger_joint1 multiplier=1.0 offset=0.0 -> joint=rg2_finger_joint1 multiplier=1 offset=0; origin xyz=0.105 -0.017 0 rpy=0 0 0 -> xyz=-0.017 0.0 0.055 rpy=0.0 -0.772 0.0; parent rg2_hand -> finger_2_origin

Commit message: Parallelgreifer - Finger zeigen noch falsch, Zwischenstand

File: urdf/ur5_rg2.urdf (robot description, URDF)
Before this commit: robot ur5_rg2, 21 links, 20 joints
Joints:
- joint gripper_bracket_joint: origin xyz=0 0 0.05 rpy=0 0 0 -> xyz=0 0.0823 0 rpy=1.570796325 0 1.570796325

Commit message: Zwischenstand - aktueller gripper_bracket_joint Stand

File: urdf/ur5_rg2.urdf (robot description, URDF)
Before this commit: robot ur5_rg2, 21 links, 20 joints
Joints:
- joint gripper_bracket_joint: origin xyz=0 0.0823 0 rpy=1.570796325 0 1.570796325 -> xyz=0 0.0823 0 rpy=1.570796325 0 0

Commit message: Parallelgreifer am Flansch - Finger zeigen seitlich, muss nach vorne

File: urdf/ur5_rg2.urdf (robot description, URDF)
Before this commit: robot ur5_rg2, 21 links, 20 joints
Joints:
- joint gripper_bracket_joint: origin xyz=0 0.0823 0 rpy=1.570796325 0 0 -> xyz=0 0.0823 0 rpy=1.570796325 0 1.570796325

Commit message: Stand vom 14.04. abends gespeichert

File: urdf/ur5_rg2.urdf (robot description, URDF)
Before this commit: robot ur5_rg2, 21 links, 20 joints
Links:
- link base_link: geometry collision mesh filename=package://ur5_rg2_ign/ur5_rg2/meshes/collision/ur5/base.stl; visual mesh filename=package://ur5_rg2_ign/ur5_rg2/meshes/visual/ur5/base.dae
- link finger_1_finger_tip: geometry collision mesh filename=package://ur5_rg2_ign/ur5_rg2/meshes/visual/rg2/finger_tip.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; visual mesh filename=package://ur5_rg2_ign/ur5_rg2/meshes/visual/rg2/finger_tip.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
- link finger_1_flex_finger: geometry collision mesh filename=package://ur5_rg2_ign/ur5_rg2/meshes/visual/rg2/flex_finger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; visual mesh filename=package://ur5_rg2_ign/ur5_rg2/meshes/visual/rg2/flex_finger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
- link finger_1_moment_arm: geometry collision mesh filename=package://ur5_rg2_ign/ur5_rg2/meshes/visual/rg2/moment_arm.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; visual mesh filename=package://ur5_rg2_ign/ur5_rg2/meshes/visual/rg2/moment_arm.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
- link finger_1_truss_arm: geometry collision mesh filename=package://ur5_rg2_ign/ur5_rg2/meshes/visual/rg2/truss_arm.s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; visual mesh filename=package://ur5_rg2_ign/ur5_rg2/meshes/visual/rg2/truss_arm.s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
- link finger_2_finger_tip: geometry collision mesh filename=package://ur5_rg2_ign/ur5_rg2/meshes/visual/rg2/finger_tip.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; visual mesh filename=package://ur5_rg2_ign/ur5_rg2/meshes/visual/rg2/finger_tip.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
- link finger_2_flex_finger: geometry collision mesh filename=package://ur5_rg2_ign/ur5_rg2/meshes/visual/rg2/flex_finger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; visual mesh filename=package://ur5_rg2_ign/ur5_rg2/meshes/visual/rg2/flex_finger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
- link finger_2_moment_arm: geometry collision mesh filename=package://ur5_rg2_ign/ur5_rg2/meshes/visual/rg2/moment_arm.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; visual mesh filename=package://ur5_rg2_ign/ur5_rg2/meshes/visual/rg2/moment_arm.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
- link finger_2_truss_arm: geometry collision mesh filename=package://ur5_rg2_ign/ur5_rg2/meshes/visual/rg2/truss_arm.s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; visual mesh filename=package://ur5_rg2_ign/ur5_rg2/meshes/visual/rg2/truss_arm.s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
- link forearm_link: geometry collision mesh filename=package://ur5_rg2_ign/ur5_rg2/meshes/collision/ur5/forearm.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; visual mesh filename=package://ur5_rg2_ign/ur5_rg2/meshes/visual/ur5/forearm.dae
- link gripper_body: geometry collision mesh filename=package://ur5_rg2_ign/ur5_rg2/meshes/visual/rg2/body.stl; visual mesh filename=package://ur5_rg2_ign/ur5_rg2/meshes/visual/rg2/body.stl
- link gripper_bracket: geometry collision mesh filename=package://ur5_rg2_ign/ur5_rg2/meshes/visual/rg2/single_brac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; visual mesh filename=package://ur5_rg2_ign/ur5_rg2/meshes/visual/rg2/single_brac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
- link shoulder_link: geometry collision mesh filename=package://ur5_rg2_ign/ur5_rg2/meshes/collision/ur5/shoulder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; visual mesh filename=package://ur5_rg2_ign/ur5_rg2/meshes/visual/ur5/shoulder.dae
- link upper_arm_link: geometry collision mesh filename=package://ur5_rg2_ign/ur5_rg2/meshes/collision/ur5/upperarm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; visual mesh filename=package://ur5_rg2_ign/ur5_rg2/meshes/visual/ur5/upperarm.dae
- link wrist_1_link: geometry collision mesh filename=package://ur5_rg2_ign/ur5_rg2/meshes/collision/ur5/wrist1.s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; visual mesh filename=package://ur5_rg2_ign/ur5_rg2/meshes/visual/ur5/wrist1.dae
- link wrist_2_link: geometry collision mesh filename=package://ur5_rg2_ign/ur5_rg2/meshes/collision/ur5/wrist2.s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; visual mesh filename=package://ur5_rg2_ign/ur5_rg2/meshes/visual/ur5/wrist2.dae
- link wrist_3_link: geometry collision mesh filename=package://ur5_rg2_ign/ur5_rg2/meshes/collision/ur5/wrist3.s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; visual mesh filename=package://ur5_rg2_ign/ur5_rg2/meshes/visual/ur5/wrist3.dae
Joints:
- joint end_effector_frame_fixed_joint: origin xyz=0 0.275 0 rpy=-1.570796325 0 0 -> xyz=0 0 -0.12 rpy=0 0 0
- joint gripper_bracket_joint: origin xyz=0 0.0823 0 rpy=-1.570796325 0 0 -> xyz=0 0 0.001 rpy=0 0 0; parent wrist_3_link -> tool0

Commit message: Fix: Mesh-Pfade auf absolute Pfade geändert - Roboter sichtbar

File: urdf/ur5_rg2.urdf (robot description, URDF)
Before this commit: robot ur5_rg2, 21 links, 20 joints
Links:
- link base_link: geometry collision mesh filename=/home/s/ros2_ws/install/ur5_rg2_ign/share/ur5_rg2_ign/ur5_r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; visual mesh filename=/home/s/ros2_ws/install/ur5_rg2_ign/share/ur5_rg2_ign/ur5_r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
- link finger_1_finger_tip: geometry collision mesh filename=/home/s/ros2_ws/install/ur5_rg2_ign/share/ur5_rg2_ign/ur5_r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; visual mesh filename=/home/s/ros2_ws/install/ur5_rg2_ign/share/ur5_rg2_ign/ur5_r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
- link finger_1_flex_finger: geometry collision mesh filename=/home/s/ros2_ws/install/ur5_rg2_ign/share/ur5_rg2_ign/ur5_r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; visual mesh filename=/home/s/ros2_ws/install/ur5_rg2_ign/share/ur5_rg2_ign/ur5_r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
- link finger_1_moment_arm: geometry collision mesh filename=/home/s/ros2_ws/install/ur5_rg2_ign/share/ur5_rg2_ign/ur5_r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; visual mesh filename=/home/s/ros2_ws/install/ur5_rg2_ign/share/ur5_rg2_ign/ur5_r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
- link finger_1_truss_arm: geometry collision mesh filename=/home/s/ros2_ws/install/ur5_rg2_ign/share/ur5_rg2_ign/ur5_r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; visual mesh filename=/home/s/ros2_ws/install/ur5_rg2_ign/share/ur5_rg2_ign/ur5_r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
- link finger_2_finger_tip: geometry collision mesh filename=/home/s/ros2_ws/install/ur5_rg2_ign/share/ur5_rg2_ign/ur5_r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; visual mesh filename=/home/s/ros2_ws/install/ur5_rg2_ign/share/ur5_rg2_ign/ur5_r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
- link finger_2_flex_finger: geometry collision mesh filename=/home/s/ros2_ws/install/ur5_rg2_ign/share/ur5_rg2_ign/ur5_r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; visual mesh filename=/home/s/ros2_ws/install/ur5_rg2_ign/share/ur5_rg2_ign/ur5_r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
- link finger_2_moment_arm: geometry collision mesh filename=/home/s/ros2_ws/install/ur5_rg2_ign/share/ur5_rg2_ign/ur5_r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; visual mesh filename=/home/s/ros2_ws/install/ur5_rg2_ign/share/ur5_rg2_ign/ur5_r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
- link finger_2_truss_arm: geometry collision mesh filename=/home/s/ros2_ws/install/ur5_rg2_ign/share/ur5_rg2_ign/ur5_r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; visual mesh filename=/home/s/ros2_ws/install/ur5_rg2_ign/share/ur5_rg2_ign/ur5_r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
- link forearm_link: geometry collision mesh filename=/home/s/ros2_ws/install/ur5_rg2_ign/share/ur5_rg2_ign/ur5_r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; visual mesh filename=/home/s/ros2_ws/install/ur5_rg2_ign/share/ur5_rg2_ign/ur5_r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
- link gripper_body: geometry collision mesh filename=/home/s/ros2_ws/install/ur5_rg2_ign/share/ur5_rg2_ign/ur5_r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; visual mesh filename=/home/s/ros2_ws/install/ur5_rg2_ign/share/ur5_rg2_ign/ur5_r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
- link gripper_bracket: geometry collision mesh filename=/home/s/ros2_ws/install/ur5_rg2_ign/share/ur5_rg2_ign/ur5_r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; visual mesh filename=/home/s/ros2_ws/install/ur5_rg2_ign/share/ur5_rg2_ign/ur5_r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
- link shoulder_link: geometry collision mesh filename=/home/s/ros2_ws/install/ur5_rg2_ign/share/ur5_rg2_ign/ur5_r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; visual mesh filename=/home/s/ros2_ws/install/ur5_rg2_ign/share/ur5_rg2_ign/ur5_r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
- link upper_arm_link: geometry collision mesh filename=/home/s/ros2_ws/install/ur5_rg2_ign/share/ur5_rg2_ign/ur5_r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; visual mesh filename=/home/s/ros2_ws/install/ur5_rg2_ign/share/ur5_rg2_ign/ur5_r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
- link wrist_1_link: geometry collision mesh filename=/home/s/ros2_ws/install/ur5_rg2_ign/share/ur5_rg2_ign/ur5_r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; visual mesh filename=/home/s/ros2_ws/install/ur5_rg2_ign/share/ur5_rg2_ign/ur5_r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
- link wrist_2_link: geometry collision mesh filename=/home/s/ros2_ws/install/ur5_rg2_ign/share/ur5_rg2_ign/ur5_r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; visual mesh filename=/home/s/ros2_ws/install/ur5_rg2_ign/share/ur5_rg2_ign/ur5_r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
- link wrist_3_link: geometry collision mesh filename=/home/s/ros2_ws/install/ur5_rg2_ign/share/ur5_rg2_ign/ur5_r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; visual mesh filename=/home/s/ros2_ws/install/ur5_rg2_ign/share/ur5_rg2_ign/ur5_r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

Commit message: Fix: Greifer korrekt am Flansch montiert - horizontal ausgerichtet

File: urdf/ur5_rg2.urdf (robot description, URDF)
Before this commit: robot ur5_rg2, 21 links, 20 joints
Joints:
- joint gripper_bracket_joint: origin xyz=0 0.0823 0 rpy=1.570796325 0 1.570796325 -> xyz=0 0.0823 0 rpy=-1.570796325 0 0
